Commit message: update

File: urdf/slam2robot.urdf (robot description, URDF)
Before this commit: robot slam2robot, 13 links, 12 joints
Links:
- link base_link: mass 2.8289 -> 3.7053
Joints:
- joint camera_optical_joint: origin xyz=0 0 0 rpy= 0 -1.5708 0 -> xyz=0 0 0 rpy=0 -1.5708 0
- joint imu_joint: origin xyz=-0.090187 0 0.035717 rpy=0 0 0 -> xyz=-0.073325 0 0.065717 rpy=0 0 0
- joint l1: origin xyz=0 0 0.075717 rpy=1.5708 -1.189 0 -> xyz=0 0 0.10072 rpy=1.5708 -1.189 0
- joint lidar_front_joint: origin xyz=0.090769 0 0.050717 rpy=0 0 0 -> xyz=0.15193 0 0.07717 rpy=0 0 0
